File: Board/Encoder_v1.brd (EAGLE design)
At the start: 89.6 x 106.3 mm, 20 parts, among them IC1 7805T, Q1 IRF620, Q2 IRF620, SW1 EC12E_SW, X1 HD44780LCD-1602

Commit message: Adição dos arquivos de layout da PCB
Parts:
- added U$3: (no value), SparkFun-Aesthetics:OSHW-LOGO-M_COPPER
- Q1, Q2: value IRF620 -> IRF640
Changed lines of the file:
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@@
 <element name="MOTOR" library="dp_devices" package="TERMINAL_BLOCK_2P_5" value="CON_TERMINAL_BLOCK_02-5MM" x="7.62" y="57.15" rot="R90"/>
 <element name="POW" library="gm-switches" package="M9040P" value="" x="67.818" y="9.398" rot="R180"/>
-<element name="Q1" library="transistor-fet" package="TO220" value="IRF620" x="24.13" y="48.26"/>
-<element name="Q2" library="transistor-fet" package="TO220" value="IRF620" x="24.13" y="19.05"/>
+<element name="Q1" library="transistor-fet" package="TO220" value="IRF640" x="24.13" y="48.26"/>
+<element name="Q2" library="transistor-fet" package="TO220" value="IRF640" x="24.13" y="19.05"/>
 <element name="R1" library="SparkFun-Passives" package="AXIAL-0.4" value="220R" x="11.43" y="6.35"/>
 <element name="R2" library="SparkFun-Passives" package="AXIAL-0.4" value="220R" x="11.43" y="38.1" rot="R180"/>
@@
 </element>
 <element name="D1" library="gm-diodes" package="DO41-4" value="1n4007" x="13.97" y="57.15" rot="R90"/>
+<element name="U$3" library="SparkFun-Aesthetics" package="OSHW-LOGO-M_COPPER" value="" x="45.974" y="84.582" rot="MR0"/>
 </elements>
 <signals>

Commit message: Minor Updates na placa, update do código, inicio da programação do encoder
Parts:
- added C1: 1000uf, SparkFun-Passives:CPOL-RADIAL-1000UF-25V
- A01: value ARDUINONANO -> ARDUINO NANO
- RV1: value (none) -> 330R
- SW1: value EC12E_SW -> Encoder
- moved IC1 3.64 mm to (83.3, 32.5)
- moved 12V 1.52 mm to (82.5, 2.79)
- moved LED2 0.25 mm to (7.87, 47.0), turned to 180 degrees
- turned LED1 to 180 degrees
- renumbered POW to POWER, U$1 to A01
Connections:
- net +12V: now also C1.1
- net N$1: now also LED1.K, R1.P$1; no longer LED2.A, R2.P$2
- net N$13: now also LED2.A; no longer LED2.K
- net N$8: now also LED2.K, R2.P$2; no longer LED1.A, R1.P$1
- net N$9: now also LED1.A; no longer LED1.K
- net SWGND: now also C1.2
Routing:
- net SWGND: track 301.4 -> 318.1 mm
- net +12V: track 181.2 -> 188.6 mm
- net N$1: track 8.89 -> 11.4 mm
- net N$8: track 11.4 -> 9.14 mm
- net N$4: track 14.1 -> 15.3 mm
Other:
- board text added: "+"
- board text added: "-"
- board text added: "TR1"

Commit message: Minor Updates na placa, update do código, inicio da programação do encoder
Parts:
- moved THERMISTOR 2.54 mm to (67.3, 20.3), turned to 180 degrees
Connections:
- net N$3: now also A01.A4; no longer A01.A0
- net N$5: now also A01.A6; no longer A01.A2
- net N$6: now also A01.A7; no longer A01.A5
- net N$7: now also A01.A5; no longer A01.A1
Routing:
- net N$3: track 48.3 -> 60.2 mm
- net N$5: track 52.2 -> 62.8 mm
- net N$7: track 51.6 -> 61.1 mm
- net SWGND: track 318.1 -> 315.8 mm
- net N$6: track 21.9 -> 22.4 mm
Other:
- board text added: "FilaEX Control Board V1.0.1 - Encoder"
- board text removed: "FilaEX Control Board V1.0 - Encoder"
Changed lines of the file:
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@@
 <wire x1="0.584" y1="102.85" x2="0.584" y2="-3.429" width="0" layer="20"/>
 <wire x1="0.584" y1="-3.429" x2="90.17" y2="-3.429" width="0" layer="20"/>
-<text x="77.724" y="93.726" size="2.1844" layer="16" font="vector" ratio="20" distance="62" rot="MR0">FilaEX Control Board V1.0 - Encoder</text>
+<text x="77.724" y="93.726" size="2.1844" layer="16" font="vector" ratio="20" distance="62" rot="MR0">FilaEX Control Board V1.0.1 - Encoder</text>
 <text x="67.818" y="89.408" size="2.1844" layer="16" font="vector" ratio="20" distance="62" rot="MR0">Design by: Raphael Toselli</text>
 <text x="75.692" y="77.724" size="2.1844" layer="16" font="vector" ratio="20" distance="62" rot="MR0">https://github.com/rtoselli/FilaExBR</text>
@@
 <element name="R3" library="SparkFun-Passives" package="AXIAL-0.4" value="47k" x="66.04" y="34.29" rot="R90"/>
 <element name="RV1" library="SparkFun-Electromechanical" package="TRIM_POT" value="330R" x="31.115" y="59.69"/>
-<element name="THERMISTOR" library="pinhead" package="1X02" value="" x="64.77" y="20.32" smashed="yes">
-<attribute name="NAME" x="60.3758" y="22.4028" size="1.27" layer="25" ratio="10"/>
-<attribute name="VALUE" x="62.23" y="17.145" size="1.27" layer="27"/>
+<element name="THERMISTOR" library="pinhead" package="1X02" value="" x="67.31" y="20.32" smashed="yes" rot="R180">
+<attribute name="NAME" x="71.7042" y="18.2372" size="1.27" layer="25" ratio="10" rot="R180"/>
+<attribute name="VALUE" x="69.85" y="23.495" size="1.27" layer="27" rot="R180"/>
 </element>
 <element name="A01" library="jet-lib" package="PDIP-32" value="ARDUINO NANO" x="39.37" y="45.72" smashed="yes"/>
@@
 <contactref element="SW1" pad="C"/>
 <contactref element="THERMISTOR" pad="1"/>
-<wire x1="63.5" y1="20.32" x2="63.5" y2="18.415" width="1.016" layer="16"/>
-<wire x1="63.5" y1="18.415" x2="67.818" y2="14.097" width="1.016" layer="16"/>
 <contactref element="X1" pad="1"/>
 <contactref element="X1" pad="5"/>
@@
 <wire x1="83.312" y1="22.352" x2="83.312" y2="15.24" width="1.016" layer="16"/>
 <wire x1="83.312" y1="15.24" x2="84.328" y2="14.224" width="1.016" layer="16"/>
+<wire x1="68.58" y1="20.32" x2="72.136" y2="20.32" width="1.016" layer="16"/>
+<wire x1="72.136" y1="20.32" x2="73.66" y2="21.844" width="1.016" layer="16"/>
 </signal>
 <signal name="N$6">
 <contactref element="R3" pad="P$1"/>
 <contactref element="THERMISTOR" pad="2"/>
-<contactref element="A01" pad="A5"/>
-<wire x1="66.04" y1="20.32" x2="66.04" y2="24.13" width="1.016" layer="16"/>
-<wire x1="66.04" y1="24.13" x2="66.04" y2="29.21" width="1.016" layer="16"/>
-<wire x1="54.61" y1="20.32" x2="55.88" y2="20.32" width="1.016" layer="16"/>
-<wire x1="55.88" y1="20.32" x2="59.69" y2="24.13" width="1.016" layer="16"/>
-<wire x1="59.69" y1="24.13" x2="66.04" y2="24.13" width="1.016" layer="16"/>
+<contactref element="A01" pad="A7"/>
+<wire x1="54.61" y1="15.24" x2="59.182" y2="15.24" width="1.016" layer="16"/>
+<wire x1="59.182" y1="15.24" x2="64.262" y2="20.32" width="1.016" layer="16"/>
+<wire x1="64.262" y1="20.32" x2="66.04" y2="20.32" width="1.016" layer="16"/>
+<wire x1="66.04" y1="29.21" x2="66.04" y2="20.32" width="1.016" layer="16"/>
 </signal>
 <signal name="+12V">
@@
 <wire x1="73.152" y1="32.258" x2="66.04" y2="39.37" width="1.016" layer="16"/>
 </signal>
-<signal name="N$3">
-<contactref element="A01" pad="A0"/>
-<contactref element="SW1" pad="E"/>
-<wire x1="54.61" y1="33.02" x2="56.896" y2="33.02" width="1.016" layer="16"/>
-<wire x1="56.896" y1="33.02" x2="59.69" y2="36.068" width="1.016" layer="16"/>
-<wire x1="59.69" y1="36.068" x2="59.69" y2="52.324" width="1.016" layer="16"/>
-<wire x1="78.715" y1="60.833" x2="81.24" y2="59.07" width="1.016" layer="16"/>
-<wire x1="59.69" y1="52.324" x2="68.199" y2="60.833" width="1.016" layer="16"/>
-<wire x1="68.199" y1="60.833" x2="78.715" y2="60.833" width="1.016" layer="16"/>
-</signal>
 <signal name="N$7">
 <contactref element="SW1" pad="A"/>
-<contactref element="A01" pad="A1"/>
-<wire x1="54.61" y1="30.48" x2="57.277" y2="30.48" width="1.016" layer="16"/>
-<wire x1="57.277" y1="30.48" x2="61.722" y2="34.671" width="1.016" layer="16"/>
-<wire x1="61.722" y1="34.671" x2="61.722" y2="51.562" width="1.016" layer="16"/>
-<wire x1="65.405" y1="55.245" x2="74.93" y2="55.245" width="1.016" layer="16"/>
+<wire x1="61.722" y1="24.892" x2="61.722" y2="50.546" width="1.016" layer="16"/>
+<wire x1="65.913" y1="55.245" x2="74.93" y2="55.245" width="1.016" layer="16"/>
 <wire x1="74.93" y1="55.245" x2="76.2" y2="53.975" width="1.016" layer="16"/>
 <wire x1="76.2" y1="53.975" x2="76.2" y2="44.61" width="1.016" layer="16"/>
 <wire x1="76.2" y1="44.61" x2="76.24" y2="44.57" width="1.016" layer="16"/>
-<wire x1="61.722" y1="51.562" x2="65.405" y2="55.245" width="1.016" layer="16"/>
+<wire x1="61.722" y1="50.546" x2="65.913" y2="55.245" width="1.016" layer="16"/>
+<contactref element="A01" pad="A5"/>
+<wire x1="61.722" y1="24.892" x2="58.674" y2="22.098" width="1.016" layer="16"/>
+<wire x1="58.674" y1="22.098" x2="56.896" y2="20.32" width="1.016" layer="16"/>
+<wire x1="56.896" y1="20.32" x2="54.61" y2="20.32" width="1.016" layer="16"/>
 </signal>
 <signal name="N$5">
 <contactref element="SW1" pad="B"/>
-<contactref element="A01" pad="A2"/>
-<wire x1="54.61" y1="27.94" x2="57.785" y2="27.94" width="1.016" layer="16"/>
-<wire x1="57.785" y1="27.94" x2="63.754" y2="33.401" width="1.016" layer="16"/>
-<wire x1="63.754" y1="33.401" x2="63.754" y2="49.022" width="1.016" layer="16"/>
+<wire x1="63.754" y1="22.86" x2="63.754" y2="49.022" width="1.016" layer="16"/>
 <wire x1="63.754" y1="49.022" x2="64.897" y2="50.165" width="1.016" layer="16"/>
 <wire x1="64.897" y1="50.165" x2="68.834" y2="50.165" width="1.016" layer="16"/>
@@
 <wire x1="81.28" y1="41.91" x2="81.28" y2="44.53" width="1.016" layer="16"/>
 <wire x1="81.28" y1="44.53" x2="81.24" y2="44.57" width="1.016" layer="16"/>
+<contactref element="A01" pad="A6"/>
+<wire x1="63.754" y1="22.86" x2="58.674" y2="17.78" width="1.016" layer="16"/>
+<wire x1="58.674" y1="17.78" x2="54.61" y2="17.78" width="1.016" layer="16"/>
 </signal>
 <signal name="N$9">
@@
 <wire x1="6.35" y1="46.99" x2="6.35" y2="38.1" width="1.016" layer="16"/>
 </signal>
+<signal name="N$3">
+<contactref element="A01" pad="A4"/>
+<contactref element="SW1" pad="E"/>
+<wire x1="81.24" y1="59.07" x2="81.24" y2="59.73" width="1.016" layer="16"/>
+<wire x1="81.24" y1="59.73" x2="78.232" y2="62.738" width="1.016" layer="16"/>
+<wire x1="78.232" y1="62.738" x2="75.184" y2="62.738" width="1.016" layer="16"/>
+<wire x1="75.184" y1="62.738" x2="69.85" y2="57.404" width="1.016" layer="16"/>
+<wire x1="69.85" y1="57.404" x2="65.024" y2="57.404" width="1.016" layer="16"/>
+<wire x1="65.024" y1="57.404" x2="59.69" y2="52.07" width="1.016" layer="16"/>
+<wire x1="59.69" y1="52.07" x2="59.69" y2="26.162" width="1.016" layer="16"/>
+<wire x1="59.69" y1="26.162" x2="56.388" y2="22.86" width="1.016" layer="16"/>
+<wire x1="56.388" y1="22.86" x2="54.61" y2="22.86" width="1.016" layer="16"/>
+</signal>
 </signals>

Commit message: Update board files and readme
Parts:
- Q1, Q2: value IRF640 -> IRLB3813
- moved FAN2 2.03 mm to (31.8, 1.78)
- moved FAN1 1.78 mm to (24.1, 2.03)
Routing:
- net +12V: track 188.6 -> 196.1 mm
- net SWGND: track 315.8 -> 322.1 mm
- net N$12: track 36.9 -> 33.0 mm
Other:
- board size 89.6 x 106.3 mm -> 90.1 x 106.8 mm
