File: Board/Encoder_v1.sch (EAGLE design)
At the start: 20 parts, among them IC1 7805T, Q1 IRF620, Q2 IRF620, SW1 EC12E_SW, X1 HD44780LCD-1602

Commit message: Adição dos arquivos de layout da PCB
Parts:
- Q1, Q2: value IRF620 -> IRF640
Changed lines of the file:
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@@
 </classes>
 <parts>
-<part name="Q1" library="transistor-fet" deviceset="IRF620" device=""/>
-<part name="Q2" library="transistor-fet" deviceset="IRF620" device=""/>
+<part name="Q1" library="transistor-fet" deviceset="IRF620" device="" value="IRF640"/>
+<part name="Q2" library="transistor-fet" deviceset="IRF620" device="" value="IRF640"/>
 <part name="12V" library="dp_devices" deviceset="CON_TERMINAL_BLOCK_02" device="-5MM"/>
 <part name="HEATER" library="dp_devices" deviceset="CON_TERMINAL_BLOCK_02" device="-5MM"/>

Commit message: Minor Updates na placa, update do código, inicio da programação do encoder
Parts:
- added C1: 1000uf, SparkFun-Passives:CAP_POLPTH4
- A01: value ARDUINONANO -> ARDUINO NANO
- RV1: value (none) -> 330R
- SW1: value EC12E_SW -> Encoder
- renumbered POW to POWER, U$1 to A01
Connections:
- net +12V: now also C1.+
- net N$1: now also LED1.C, R1.1; no longer LED2.A, R2.2
- net N$13: now also LED2.A; no longer LED2.C
- net N$8: now also LED2.C, R2.2; no longer LED1.A, R1.1
- net N$9: now also LED1.A; no longer LED1.C
- net SWGND: now also C1.-
Other:
- moved on the sheet: LED1, LED2
Changed lines of the file:
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@@
 <part name="IC1" library="adafruit" deviceset="78*" device="T" technology="05"/>
 <part name="X1" library="adafruit" deviceset="HD44780LCD" device="-1602"/>
-<part name="RV1" library="SparkFun-Electromechanical" deviceset="POT" device="TRIM"/>
-<part name="POW" library="gm-switches" deviceset="SPDT" device=""/>
-<part name="U$1" library="jet-lib" deviceset="ARDUINONANO" device=""/>
+<part name="RV1" library="SparkFun-Electromechanical" deviceset="POT" device="TRIM" value="330R"/>
+<part name="POWER" library="gm-switches" deviceset="SPDT" device=""/>
+<part name="A01" library="jet-lib" deviceset="ARDUINONANO" device="" value="ARDUINO NANO"/>
 <part name="R3" library="SparkFun-Passives" deviceset="RESISTOR" device="PTH-1/4W" value="47k"/>
-<part name="SW1" library="switch-alps" deviceset="EC12E_SW" device=""/>
+<part name="SW1" library="switch-alps" deviceset="EC12E_SW" device="" value="Encoder"/>
 <part name="D1" library="gm-diodes" deviceset="1N400X" device=".4" value="1n4007"/>
+<part name="C1" library="SparkFun-Passives" deviceset="CAP_POL" device="PTH4" value="1000uf"/>
 </parts>
 <sheets>
@@
 <instance part="FAN1" gate="G$1" x="-10.16" y="22.86" rot="R180"/>
 <instance part="FAN2" gate="G$1" x="-10.16" y="7.62" rot="R180"/>
-<instance part="LED1" gate="G$1" x="48.26" y="22.86" rot="R180"/>
-<instance part="LED2" gate="G$1" x="66.04" y="22.86" rot="R180"/>
+<instance part="LED1" gate="G$1" x="48.26" y="27.94"/>
+<instance part="LED2" gate="G$1" x="66.04" y="27.94"/>
 <instance part="R1" gate="G$1" x="48.26" y="12.7" rot="R270"/>
 <instance part="R2" gate="G$1" x="66.04" y="12.7" rot="R90"/>
@@
 <instance part="X1" gate="G$1" x="111.76" y="-22.86"/>
 <instance part="RV1" gate="G$1" x="93.98" y="10.16" rot="R270"/>
-<instance part="POW" gate="1" x="2.54" y="83.82" rot="R270"/>
-<instance part="U$1" gate="G$1" x="88.9" y="104.14"/>
+<instance part="POWER" gate="1" x="2.54" y="83.82" rot="R270"/>
+<instance part="A01" gate="G$1" x="88.9" y="104.14"/>
 <instance part="R3" gate="G$1" x="137.16" y="86.36" rot="R180"/>
 <instance part="SW1" gate="G$1" x="160.02" y="111.76"/>
 <instance part="SW1" gate="G$2" x="157.48" y="81.28"/>
 <instance part="D1" gate="1" x="5.08" y="58.42" rot="R90"/>
+<instance part="C1" gate="G$1" x="12.7" y="81.28"/>
 </instances>
 <busses>
 </busses>
 <nets>
-<net name="N$1" class="0">
-<segment>
-<pinref part="LED2" gate="G$1" pin="A"/>
-<pinref part="R2" gate="G$1" pin="2"/>
-<wire x1="66.04" y1="17.78" x2="66.04" y2="20.32" width="0.1524" layer="91"/>
-</segment>
-</net>
 <net name="N$2" class="0">
 <segment>
@@
 <segment>
 <pinref part="IC1" gate="A1" pin="GND"/>
-<pinref part="POW" gate="1" pin="S"/>
-<wire x1="30.48" y1="76.2" x2="7.62" y2="76.2" width="0.1524" layer="91"/>
+<pinref part="POWER" gate="1" pin="S"/>
+<wire x1="30.48" y1="76.2" x2="12.7" y2="76.2" width="0.1524" layer="91"/>
+<wire x1="12.7" y1="76.2" x2="7.62" y2="76.2" width="0.1524" layer="91"/>
 <wire x1="7.62" y1="76.2" x2="7.62" y2="78.74" width="0.1524" layer="91"/>
+<pinref part="C1" gate="G$1" pin="-"/>
+<junction x="12.7" y="76.2"/>
 </segment>
 <segment>
@@
 </segment>
 <segment>
-<pinref part="U$1" gate="G$1" pin="GND"/>
+<pinref part="A01" gate="G$1" pin="GND"/>
 <wire x1="83.82" y1="86.36" x2="78.74" y2="86.36" width="0.1524" layer="91"/>
 <label x="78.74" y="86.36" size="1.778" layer="95" rot="R180" xref="yes"/>
@@
 <pinref part="THERMISTOR" gate="G$1" pin="2"/>
 <wire x1="137.16" y1="55.88" x2="142.24" y2="55.88" width="0.1524" layer="91"/>
-<pinref part="U$1" gate="G$1" pin="A5"/>
+<pinref part="A01" gate="G$1" pin="A5"/>
 <wire x1="137.16" y1="55.88" x2="114.3" y2="55.88" width="0.1524" layer="91"/>
 <junction x="137.16" y="55.88"/>
@@
 <pinref part="IC1" gate="A1" pin="VI"/>
 <wire x1="-2.54" y1="86.36" x2="0" y2="86.36" width="0.1524" layer="91"/>
-<wire x1="0" y1="86.36" x2="20.32" y2="86.36" width="0.1524" layer="91"/>
+<wire x1="0" y1="86.36" x2="12.7" y2="86.36" width="0.1524" layer="91"/>
+<wire x1="12.7" y1="86.36" x2="20.32" y2="86.36" width="0.1524" layer="91"/>
 <wire x1="20.32" y1="86.36" x2="20.32" y2="83.82" width="0.1524" layer="91"/>
 <label x="20.32" y="86.36" size="1.778" layer="95" rot="R90" xref="yes"/>
@@
 <pinref part="FAN2" gate="G$1" pin="2"/>
 <pinref part="FAN1" gate="G$1" pin="2"/>
+<pinref part="C1" gate="G$1" pin="+"/>
+<wire x1="12.7" y1="86.36" x2="12.7" y2="83.82" width="0.1524" layer="91"/>
+<junction x="12.7" y="86.36"/>
 </segment>
 <segment>
@@
 </segment>
 <segment>
-<pinref part="U$1" gate="G$1" pin="+5V"/>
+<pinref part="A01" gate="G$1" pin="+5V"/>
 <pinref part="R3" gate="G$1" pin="2"/>
 <wire x1="132.08" y1="86.36" x2="114.3" y2="86.36" width="0.1524" layer="91"/>
@@
 <net name="N$3" class="0">
 <segment>
-<pinref part="U$1" gate="G$1" pin="A0"/>
+<pinref part="A01" gate="G$1" pin="A0"/>
 <pinref part="SW1" gate="G$2" pin="2"/>
 <wire x1="114.3" y1="81.28" x2="152.4" y2="81.28" width="0.1524" layer="91"/>
@@
 <wire x1="157.48" y1="119.38" x2="119.38" y2="119.38" width="0.1524" layer="91"/>
 <wire x1="119.38" y1="119.38" x2="119.38" y2="76.2" width="0.1524" layer="91"/>
-<pinref part="U$1" gate="G$1" pin="A1"/>
+<pinref part="A01" gate="G$1" pin="A1"/>
 <wire x1="114.3" y1="76.2" x2="119.38" y2="76.2" width="0.1524" layer="91"/>
 </segment>
@@
 <wire x1="162.56" y1="124.46" x2="121.92" y2="124.46" width="0.1524" layer="91"/>
 <wire x1="121.92" y1="124.46" x2="121.92" y2="71.12" width="0.1524" layer="91"/>
-<pinref part="U$1" gate="G$1" pin="A2"/>
+<pinref part="A01" gate="G$1" pin="A2"/>
 <wire x1="121.92" y1="71.12" x2="114.3" y2="71.12" width="0.1524" layer="91"/>
 </segment>
 </net>
-<net name="N$8" class="0">
-<segment>
-<pinref part="LED1" gate="G$1" pin="A"/>
-<pinref part="R1" gate="G$1" pin="1"/>
-<wire x1="48.26" y1="20.32" x2="48.26" y2="17.78" width="0.1524" layer="91"/>
-</segment>
-</net>
 <net name="N$9" class="0">
 <segment>
 <pinref part="Q2" gate="G$1" pin="G"/>
-<pinref part="LED1" gate="G$1" pin="C"/>
-<wire x1="48.26" y1="27.94" x2="48.26" y2="33.02" width="0.1524" layer="91"/>
 <wire x1="48.26" y1="33.02" x2="48.26" y2="35.56" width="0.1524" layer="91"/>
 <wire x1="53.34" y1="66.04" x2="53.34" y2="33.02" width="0.1524" layer="91"/>
 <wire x1="53.34" y1="33.02" x2="48.26" y2="33.02" width="0.1524" layer="91"/>
+<pinref part="A01" gate="G$1" pin="D5"/>
+<wire x1="83.82" y1="66.04" x2="53.34" y2="66.04" width="0.1524" layer="91"/>
+<pinref part="LED1" gate="G$1" pin="A"/>
+<wire x1="48.26" y1="33.02" x2="48.26" y2="30.48" width="0.1524" layer="91"/>
 <junction x="48.26" y="33.02"/>
-<pinref part="U$1" gate="G$1" pin="D5"/>
-<wire x1="83.82" y1="66.04" x2="53.34" y2="66.04" width="0.1524" layer="91"/>
 </segment>
 </net>
@@
 <segment>
 <wire x1="71.12" y1="76.2" x2="71.12" y2="33.02" width="0.1524" layer="91"/>
-<pinref part="LED2" gate="G$1" pin="C"/>
 <pinref part="Q1" gate="G$1" pin="G"/>
 <wire x1="66.04" y1="35.56" x2="66.04" y2="33.02" width="0.1524" layer="91"/>
-<wire x1="66.04" y1="33.02" x2="66.04" y2="27.94" width="0.1524" layer="91"/>
 <wire x1="71.12" y1="33.02" x2="66.04" y2="33.02" width="0.1524" layer="91"/>
+<pinref part="A01" gate="G$1" pin="D3"/>
+<wire x1="71.12" y1="76.2" x2="83.82" y2="76.2" width="0.1524" layer="91"/>
+<pinref part="LED2" gate="G$1" pin="A"/>
+<wire x1="66.04" y1="33.02" x2="66.04" y2="30.48" width="0.1524" layer="91"/>
 <junction x="66.04" y="33.02"/>
-<pinref part="U$1" gate="G$1" pin="D3"/>
-<wire x1="71.12" y1="76.2" x2="83.82" y2="76.2" width="0.1524" layer="91"/>
 </segment>
 </net>
@@
 <segment>
 <pinref part="12V" gate="CON" pin="1"/>
-<pinref part="POW" gate="1" pin="P"/>
+<pinref part="POWER" gate="1" pin="P"/>
 <wire x1="-7.62" y1="81.28" x2="-2.54" y2="81.28" width="0.1524" layer="91"/>
 </segment>
@@
 <net name="N$10" class="0">
 <segment>
-<pinref part="U$1" gate="G$1" pin="D6"/>
+<pinref part="A01" gate="G$1" pin="D6"/>
 <wire x1="83.82" y1="60.96" x2="78.74" y2="60.96" width="0.1524" layer="91"/>
 <wire x1="78.74" y1="60.96" x2="78.74" y2="22.86" width="0.1524" layer="91"/>
@@
 <net name="N$11" class="0">
 <segment>
-<pinref part="U$1" gate="G$1" pin="D7"/>
+<pinref part="A01" gate="G$1" pin="D7"/>
 <wire x1="83.82" y1="55.88" x2="76.2" y2="55.88" width="0.1524" layer="91"/>
 <wire x1="76.2" y1="55.88" x2="76.2" y2="20.32" width="0.1524" layer="91"/>
@@
 <net name="N$14" class="0">
 <segment>
-<pinref part="U$1" gate="G$1" pin="D8"/>
+<pinref part="A01" gate="G$1" pin="D8"/>
 <wire x1="83.82" y1="50.8" x2="73.66" y2="50.8" width="0.1524" layer="91"/>
 <wire x1="73.66" y1="50.8" x2="73.66" y2="17.78" width="0.1524" layer="91"/>
@@
 <net name="N$15" class="0">
 <segment>
-<pinref part="U$1" gate="G$1" pin="D9"/>
+<pinref part="A01" gate="G$1" pin="D9"/>
 <wire x1="83.82" y1="45.72" x2="81.28" y2="45.72" width="0.1524" layer="91"/>
 <wire x1="81.28" y1="45.72" x2="81.28" y2="15.24" width="0.1524" layer="91"/>
@@
 <net name="N$17" class="0">
 <segment>
-<pinref part="U$1" gate="G$1" pin="D11"/>
+<pinref part="A01" gate="G$1" pin="D11"/>
 <wire x1="83.82" y1="35.56" x2="104.14" y2="35.56" width="0.1524" layer="91"/>
 <wire x1="104.14" y1="35.56" x2="104.14" y2="-2.54" width="0.1524" layer="91"/>
@@
 <net name="N$18" class="0">
 <segment>
-<pinref part="U$1" gate="G$1" pin="D12"/>
+<pinref part="A01" gate="G$1" pin="D12"/>
 <pinref part="X1" gate="G$1" pin="RS"/>
 <wire x1="83.82" y1="30.48" x2="96.52" y2="30.48" width="0.1524" layer="91"/>
@@
 </segment>
 </net>
+<net name="N$1" class="0">
+<segment>
+<pinref part="LED1" gate="G$1" pin="C"/>
+<pinref part="R1" gate="G$1" pin="1"/>
+<wire x1="48.26" y1="22.86" x2="48.26" y2="17.78" width="0.1524" layer="91"/>
+</segment>
+</net>
+<net name="N$8" class="0">
+<segment>
+<pinref part="LED2" gate="G$1" pin="C"/>
+<pinref part="R2" gate="G$1" pin="2"/>
+<wire x1="66.04" y1="22.86" x2="66.04" y2="17.78" width="0.1524" layer="91"/>
+</segment>
+</net>

Commit message: Minor Updates na placa, update do código, inicio da programação do encoder
Connections:
- net N$3: now also A01.A4; no longer A01.A0
- net N$5: now also A01.A6; no longer A01.A2
- net N$6: now also A01.A7; no longer A01.A5
- net N$7: now also A01.A5; no longer A01.A1
Other:
- note added: "The library that i used to connect the nano has the analog pins reversed! Be carefull!"
Changed lines of the file:
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@@
 <sheet>
 <plain>
+<text x="66.04" y="129.54" size="1.778" layer="91">The library that i used to connect the nano has the analog pins reversed! Be carefull!</text>
 </plain>
 <instances>
@@
 <pinref part="THERMISTOR" gate="G$1" pin="2"/>
 <wire x1="137.16" y1="55.88" x2="142.24" y2="55.88" width="0.1524" layer="91"/>
-<pinref part="A01" gate="G$1" pin="A5"/>
-<wire x1="137.16" y1="55.88" x2="114.3" y2="55.88" width="0.1524" layer="91"/>
-<junction x="137.16" y="55.88"/>
+<wire x1="142.24" y1="55.88" x2="124.46" y2="55.88" width="0.1524" layer="91"/>
+<wire x1="124.46" y1="55.88" x2="124.46" y2="45.72" width="0.1524" layer="91"/>
+<junction x="142.24" y="55.88"/>
+<pinref part="A01" gate="G$1" pin="A7"/>
+<wire x1="124.46" y1="45.72" x2="114.3" y2="45.72" width="0.1524" layer="91"/>
 </segment>
 </net>
@@
 </segment>
 </net>
-<net name="N$3" class="0">
-<segment>
-<pinref part="A01" gate="G$1" pin="A0"/>
-<pinref part="SW1" gate="G$2" pin="2"/>
-<wire x1="114.3" y1="81.28" x2="152.4" y2="81.28" width="0.1524" layer="91"/>
-</segment>
-</net>
 <net name="N$7" class="0">
 <segment>
 <pinref part="SW1" gate="G$1" pin="A"/>
-<wire x1="157.48" y1="119.38" x2="119.38" y2="119.38" width="0.1524" layer="91"/>
-<wire x1="119.38" y1="119.38" x2="119.38" y2="76.2" width="0.1524" layer="91"/>
-<pinref part="A01" gate="G$1" pin="A1"/>
-<wire x1="114.3" y1="76.2" x2="119.38" y2="76.2" width="0.1524" layer="91"/>
+<wire x1="157.48" y1="119.38" x2="116.84" y2="119.38" width="0.1524" layer="91"/>
+<pinref part="A01" gate="G$1" pin="A5"/>
+<wire x1="114.3" y1="55.88" x2="116.84" y2="55.88" width="0.1524" layer="91"/>
+<wire x1="116.84" y1="119.38" x2="116.84" y2="55.88" width="0.1524" layer="91"/>
 </segment>
 </net>
@@
 <pinref part="SW1" gate="G$1" pin="B"/>
 <wire x1="162.56" y1="119.38" x2="162.56" y2="124.46" width="0.1524" layer="91"/>
-<wire x1="162.56" y1="124.46" x2="121.92" y2="124.46" width="0.1524" layer="91"/>
-<wire x1="121.92" y1="124.46" x2="121.92" y2="71.12" width="0.1524" layer="91"/>
-<pinref part="A01" gate="G$1" pin="A2"/>
-<wire x1="121.92" y1="71.12" x2="114.3" y2="71.12" width="0.1524" layer="91"/>
+<pinref part="A01" gate="G$1" pin="A6"/>
+<wire x1="119.38" y1="50.8" x2="114.3" y2="50.8" width="0.1524" layer="91"/>
+<wire x1="162.56" y1="124.46" x2="119.38" y2="124.46" width="0.1524" layer="91"/>
+<wire x1="119.38" y1="124.46" x2="119.38" y2="50.8" width="0.1524" layer="91"/>
 </segment>
 </net>
@@
 </segment>
 </net>
+<net name="N$3" class="0">
+<segment>
+<pinref part="A01" gate="G$1" pin="A4"/>
+<wire x1="114.3" y1="60.96" x2="129.54" y2="60.96" width="0.1524" layer="91"/>
+<wire x1="129.54" y1="60.96" x2="129.54" y2="81.28" width="0.1524" layer="91"/>
+<pinref part="SW1" gate="G$2" pin="2"/>
+<wire x1="129.54" y1="81.28" x2="152.4" y2="81.28" width="0.1524" layer="91"/>
+</segment>
+</net>

Commit message: Update board files and readme
Parts:
- Q1, Q2: value IRF640 -> IRLB3813
Changed lines of the file:
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@@
 </classes>
 <parts>
-<part name="Q1" library="transistor-fet" deviceset="IRF620" device="" value="IRF640"/>
-<part name="Q2" library="transistor-fet" deviceset="IRF620" device="" value="IRF640"/>
+<part name="Q1" library="transistor-fet" deviceset="IRF620" device="" value="IRLB3813"/>
+<part name="Q2" library="transistor-fet" deviceset="IRF620" device="" value="IRLB3813"/>
 <part name="12V" library="dp_devices" deviceset="CON_TERMINAL_BLOCK_02" device="-5MM"/>
 <part name="HEATER" library="dp_devices" deviceset="CON_TERMINAL_BLOCK_02" device="-5MM"/>
